Commit message: fix: Change robot chassis offset to display right in RViz

File: Project3_AEMC/packages/my_robot/urdf/my_robot.xacro (robot description, xacro)
@@ -12,5 +12,5 @@
   <!-- Base Imaginary Fixed Joint -->
   <joint name="robot_footprint_joint" type="fixed">
-    <origin xyz="0 0 0" rpy="0 0 0" />
+    <origin xyz="0 0 0.1" rpy="0 0 0" />
     <parent link="robot_footprint"/>
     <child link="chassis" />
